Commit message: objects

File: roboschool/roboschool/models_robot/kuka_gripper_description/urdf/shelf.urdf (robot description, URDF)
Before this commit: robot table, 1 links, 0 joints
Links:
- removed link table
- added link shelf, mass 0.0; collision mesh filename=package://kuka_gripper_description/meshes/shelf.obj; visual mesh filename=package://kuka_gripper_description/meshes/shelf.obj
