Commit message: kuka urdf

File: realcomp/data/kuka_gripper_description/urdf/kuka_gripper.urdf (robot description, URDF)
Before this commit: robot kuka_gripper, 13 links, 12 joints
Joints:
- joint base_to_finger00_joint: origin xyz=0.043510971786833857 0 0 rpy=0 0 0 -> xyz=0.023510971786833857 0 0 rpy=0 0 0
- joint base_to_finger10_joint: origin xyz=-0.043510971786833857 0 0 rpy=0 0 3.141592653589793 -> xyz=-0.023510971786833857 0 0 rpy=0 0 3.141592653589793

Commit message: modified gripper

File: realcomp/data/kuka_gripper_description/urdf/kuka_gripper.urdf (robot description, URDF)
Before this commit: robot kuka_gripper, 13 links, 12 joints
Links:
- link finger_00: geometry collision mesh filename=package://kuka_gripper_description/meshes/finger_0.obj scale=1 0.7 0.7; visual mesh filename=package://kuka_gripper_description/meshes/finger_0.obj scale=1 0.7 0.7
- link finger_01: geometry collision mesh filename=package://kuka_gripper_description/meshes/finger_1.obj scale=1 0.7 0.7; visual mesh filename=package://kuka_gripper_description/meshes/finger_1.obj scale=1 0.7 0.7
- link finger_10: geometry collision mesh filename=package://kuka_gripper_description/meshes/finger_0.obj scale=1 0.7 0.7; visual mesh filename=package://kuka_gripper_description/meshes/finger_0.obj scale=1 0.7 0.7
- link finger_11: geometry collision mesh filename=package://kuka_gripper_description/meshes/finger_1.obj scale=1 0.7 0.7; visual mesh filename=package://kuka_gripper_description/meshes/finger_1.obj scale=1 0.7 0.7
Joints:
- joint finger00_to_finger01_joint: origin xyz=0 0 0.109717868338558 rpy=0 0 0 -> xyz=0 0  0.0768025078369906 rpy=0 0 0
- joint finger10_to_finger11_joint: origin xyz=0 0 0.109717868338558 rpy=0 0 0 -> xyz=0 0 0.0768025078369906 rpy=0 0 0

Commit message: skin

File: realcomp/data/kuka_gripper_description/urdf/kuka_gripper.urdf (robot description, URDF)
Before this commit: robot kuka_gripper, 13 links, 12 joints
Links:
- added link skin_00, mass 2.0; collision mesh filename=package://kuka_gripper_description/meshes/skin_0.obj scale=1 0.7 0.7; visual mesh filename=package://kuka_gripper_description/meshes/skin_0.obj scale=1 0.7 0.7
- added link skin_01, mass 2.0; collision mesh filename=package://kuka_gripper_description/meshes/skin_0.obj scale=1 0.7 0.3; visual mesh filename=package://kuka_gripper_description/meshes/skin_0.obj scale=1 0.7 0.3
- added link skin_10, mass 2.0; collision mesh filename=package://kuka_gripper_description/meshes/skin_0.obj scale=1 0.7 0.7; visual mesh filename=package://kuka_gripper_description/meshes/skin_0.obj scale=1 0.7 0.7
- added link skin_11, mass 2.0; collision mesh filename=package://kuka_gripper_description/meshes/skin_0.obj scale=1 0.7 0.3; visual mesh filename=package://kuka_gripper_description/meshes/skin_0.obj scale=1 0.7 0.3
Joints:
- added joint finger00_to_skin_joint: type fixed, parent finger_00, child skin_00, origin xyz=-0.011 0 0.045 rpy=0 0 -3
- added joint finger01_to_skin_joint: type fixed, parent finger_01, child skin_01, origin xyz=-0.013 0 0.045 rpy=0 0 -3
- added joint finger10_to_skin_joint: type fixed, parent finger_10, child skin_10, origin xyz=-0.011 0 0.045 rpy=0 0 3
- added joint finger11_to_skin_joint: type fixed, parent finger_11, child skin_11, origin xyz=-0.013 0 0.045 rpy=0 0 -3

Commit message: modified skin

File: realcomp/data/kuka_gripper_description/urdf/kuka_gripper.urdf (robot description, URDF)
Before this commit: robot kuka_gripper, 17 links, 16 joints
Links:
- link skin_00: geometry collision mesh filename=package://kuka_gripper_description/meshes/skin_0.obj scale=1 0.3 0.7; visual mesh filename=package://kuka_gripper_description/meshes/skin_0.obj scale=1 0.3 0.7
- link skin_01: geometry collision mesh filename=package://kuka_gripper_description/meshes/skin_0.obj scale=1 0.3 0.3; visual mesh filename=package://kuka_gripper_description/meshes/skin_0.obj scale=1 0.3 0.3
- link skin_10: geometry collision mesh filename=package://kuka_gripper_description/meshes/skin_0.obj scale=1 0.3 0.7; visual mesh filename=package://kuka_gripper_description/meshes/skin_0.obj scale=1 0.3 0.7
- link skin_11: geometry collision mesh filename=package://kuka_gripper_description/meshes/skin_0.obj scale=1 0.3 0.3; visual mesh filename=package://kuka_gripper_description/meshes/skin_0.obj scale=1 0.3 0.3

Commit message: 0-mass to skin

File: realcomp/data/kuka_gripper_description/urdf/kuka_gripper.urdf (robot description, URDF)
Before this commit: robot kuka_gripper, 17 links, 16 joints
Links:
- link skin_00: mass 2.0 -> 0.0
- link skin_01: mass 2.0 -> 0.0
- link skin_10: mass 2.0 -> 0.0
- link skin_11: mass 2.0 -> 0.0
