Commit message: object masses

File: realcomp/data/kuka_gripper_description/urdf/mustard.urdf (robot description, URDF)
Before this commit: robot mustard, 1 links, 0 joints
Links:
- link mustard: mass 0.2 -> 2.0

File: realcomp/data/kuka_gripper_description/urdf/tomato.urdf (robot description, URDF)
Before this commit: robot tomato, 1 links, 0 joints
Links:
- link tomato: mass 0.2 -> 3.0

Commit message: objects

File: realcomp/data/kuka_gripper_description/urdf/mustard.urdf (robot description, URDF)
Before this commit: robot mustard, 1 links, 0 joints
Links:
- link mustard: mass 2.0 -> 0.5

File: realcomp/data/kuka_gripper_description/urdf/orange.urdf (robot description, URDF)
Before this commit: robot orange, 1 links, 0 joints
Links:
- link orange: mass 0.2 -> 0.5

Commit message: objects

File: realcomp/data/kuka_gripper_description/urdf/mustard.urdf (robot description, URDF)
Before this commit: robot mustard, 1 links, 0 joints
Links:
- link mustard: mass 0.5 -> 2.0

File: realcomp/data/kuka_gripper_description/urdf/orange.urdf (robot description, URDF)
Before this commit: robot orange, 1 links, 0 joints
Links:
- link orange: mass 0.5 -> 1.5
